File: KiCad project/BatBot/BatBot.sch (KiCad schematic (older format))
At the start: 56 parts, among them J1 54550-1271, U1 STM32F439ZIYx, U2 nRF24L01P, U3 MPU-9250, U4 LM1117MPX-3_3_NOPB, X1 NX3225GD-8MHZ-STD-CRA-3, X2 XRCHA16M000F0A01R0

Commit message: finished draft board design, updated schematic
Parts:
- ANT1: symbol AMCA31-2R450G-S1F-T3:AMCA31-2R450G-S1F-T3 -> BatBot-rescue:AMCA31-2R450G-S1F-T3-AMCA31-2R450G-S1F-T3
- C1: symbol GCJ21BR71A106KE01L:GCJ21BR71A106KE01L -> BatBot-rescue:GCJ21BR71A106KE01L-GCJ21BR71A106KE01L
- C10, C11, C12, C13, C14, C15, C18, C3, C4, C5, C6, C7, C8, C9: symbol GCE21BR71H104KA01L:GCE21BR71H104KA01L -> BatBot-rescue:GCE21BR71H104KA01L-GCE21BR71H104KA01L
- C16, C24, C32: symbol 06035C103MAT2A:06035C103MAT2A -> BatBot-rescue:06035C103MAT2A-06035C103MAT2A
- C17: symbol GCM21BR11E105KA42L:GCM21BR11E105KA42L -> BatBot-rescue:GCM21BR11E105KA42L-GCM21BR11E105KA42L
- C19, C20: symbol GRM188C71E225KE11J:GRM188C71E225KE11J -> BatBot-rescue:GRM188C71E225KE11J-GRM188C71E225KE11J
- C2: symbol CL31A107MQHNNNE:CL31A107MQHNNNE -> BatBot-rescue:CL31A107MQHNNNE-CL31A107MQHNNNE
- C21, C22, C28, C29: symbol GRM0335C1H8R0DA01D:GRM0335C1H8R0DA01D -> BatBot-rescue:GRM0335C1H8R0DA01D-GRM0335C1H8R0DA01D
- C23: symbol 06035C333KAT2A:06035C333KAT2A -> BatBot-rescue:06035C333KAT2A-06035C333KAT2A
- C25: symbol 0402ZC102KAT2A:0402ZC102KAT2A -> BatBot-rescue:0402ZC102KAT2A-0402ZC102KAT2A
- C26: symbol CC0603BRNPO0BN4R7:CC0603BRNPO0BN4R7 -> BatBot-rescue:CC0603BRNPO0BN4R7-CC0603BRNPO0BN4R7
- C27: symbol EMK212B7225MG-T:EMK212B7225MG-T -> BatBot-rescue:EMK212B7225MG-T-EMK212B7225MG-T
- C30: symbol AC0402BRNPO9BN1R5:AC0402BRNPO9BN1R5 -> BatBot-rescue:AC0402BRNPO9BN1R5-AC0402BRNPO9BN1R5
- C31: symbol CC0603CRNPO8BN1R0:CC0603CRNPO8BN1R0 -> BatBot-rescue:CC0603CRNPO8BN1R0-CC0603CRNPO8BN1R0
- C33, C34: symbol 0805YC104K4Z4A:0805YC104K4Z4A -> BatBot-rescue:0805YC104K4Z4A-0805YC104K4Z4A
- D1, D2, D3: symbol dk_LED-Indication-Discrete:LTST-C190KRKT -> BatBot-rescue:LTST-C190KRKT-dk_LED-Indication-Discrete
- J1: symbol eec:54550-1271 -> BatBot-rescue:54550-1271-eec
- L1: symbol CE201210-8N2J:CE201210-8N2J -> BatBot-rescue:CE201210-8N2J-CE201210-8N2J
- L2: symbol AQ1052N7S-T:AQ1052N7S-T -> BatBot-rescue:AQ1052N7S-T-AQ1052N7S-T
- L3: symbol AIMC-0805-3N9S-T:AIMC-0805-3N9S-T -> BatBot-rescue:AIMC-0805-3N9S-T-AIMC-0805-3N9S-T
- R1, R4, R6: symbol 1-1622826-8:1-1622826-8 -> BatBot-rescue:1-1622826-8-1-1622826-8
- R2, R5: symbol 8-1676481-3:8-1676481-3 -> BatBot-rescue:8-1676481-3-8-1676481-3
- R3: symbol 2020-09-26_23-31-02:RC0201FR-07100RL -> BatBot-rescue:RC0201FR-07100RL-2020-09-26_23-31-02
- R7: symbol CRG0402F1M0:CRG0402F1M0 -> BatBot-rescue:CRG0402F1M0-CRG0402F1M0
- S1: symbol FSM8JH:FSM8JH -> BatBot-rescue:FSM8JH-FSM8JH
- U1: symbol MCU_ST_STM32F4:STM32F439ZIYx -> BatBot-rescue:STM32F439ZIYx-MCU_ST_STM32F4
- U2: symbol RF:nRF24L01P -> BatBot-rescue:nRF24L01P-RF
- U3: symbol Sensor_Motion:MPU-9250 -> BatBot-rescue:MPU-9250-Sensor_Motion
- U4: symbol dk_PMIC-Voltage-Regulators-Linear:LM1117MPX-3_3_NOPB -> BatBot-rescue:LM1117MPX-3_3_NOPB-dk_PMIC-Voltage-Regulators-Linear
- X1: symbol dk_Crystals:NX3225GD-8MHZ-STD-CRA-3 -> BatBot-rescue:NX3225GD-8MHZ-STD-CRA-3-dk_Crystals
- X2: symbol XRCHA16M000F0A01R0:XRCHA16M000F0A01R0 -> BatBot-rescue:XRCHA16M000F0A01R0-XRCHA16M000F0A01R0
Connections:
- net GND: now also C10.2, C11.2, C12.2, C13.2, C14.2, C15.2
